File: Termin_2/schematics/pull-up_down.kicad_sch (KiCad schematic)
At the start: 4 parts, among them SW1 SW_Push, SW2 SW_Push

Commit message: Added values to pull-up pull-down resistors
Parts:
- R1, R2: value R -> 10 k
Changed lines of the file:
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@@
 			)
 		)
-		(property "Value" "R"
+		(property "Value" "10 k"
 			(at 45.72 45.7199 0)
 			(effects
@@
 			)
 		)
-		(property "Value" "R"
+		(property "Value" "10 k"
 			(at 81.28 35.5599 0)
 			(effects
